Commit message: update dg5f

File: dg5f/dg5f_left_short.urdf (robot description, URDF)
Before this commit: robot dg5f_left_short, 28 links, 27 joints
Links:
- link ll_dg_1_1: mass 0.045 -> 0.0482
- link ll_dg_1_2: mass 0.025 -> 0.0164
- link ll_dg_1_3: mass 0.045 -> 0.0362
- link ll_dg_1_4: mass 0.045 -> 0.0505
- link ll_dg_2_1: mass 0.045 -> 0.0546
- link ll_dg_2_2: mass 0.045 -> 0.0362
- link ll_dg_2_3: mass 0.045 -> 0.0362
- link ll_dg_2_4: mass 0.025 -> 0.0266
- link ll_dg_3_1: mass 0.045 -> 0.0526
- link ll_dg_3_2: mass 0.045 -> 0.0362
- link ll_dg_3_3: mass 0.045 -> 0.0362
- link ll_dg_3_4: mass 0.025 -> 0.0266
- link ll_dg_4_1: mass 0.045 -> 0.0548
- link ll_dg_4_2: mass 0.045 -> 0.0362
- link ll_dg_4_3: mass 0.045 -> 0.0362
- link ll_dg_4_4: mass 0.025 -> 0.0266
- link ll_dg_5_1: mass 0.055 -> 0.0744
- link ll_dg_5_2: mass 0.025 -> 0.0164
- link ll_dg_5_3: mass 0.045 -> 0.0362
- link ll_dg_5_4: mass 0.045 -> 0.0505
- link ll_dg_palm: mass 0.35 -> 0.4007
Joints:
- joint lj_dg_base: origin xyz=0 0 0.004 rpy=0 0 0 -> xyz=0 0 0.0045 rpy=0 0 0
- joint lj_dg_palm: origin xyz=0 0 0.0698 rpy=0 0 0 -> xyz=0 0 0.022 rpy=0 0 0

File: dg5f/dg5f_right_short.urdf (robot description, URDF)
Before this commit: robot dg5f_right_short, 28 links, 27 joints
Joints:
- joint rj_dg_base: origin xyz=0 0 0.004 rpy=0 0 0 -> xyz=0 0 0.0045 rpy=0 0 0
- joint rj_dg_palm: origin xyz=0 0 0.0698 rpy=0 0 0 -> xyz=0 0 0.022 rpy=0 0 0
