Commit message: dg5f urdf modified

File: dg5f/dg5f_left.urdf (robot description, URDF)
Before this commit: robot dg5f_left, 28 links, 27 joints
Links:
- link ll_dg_1_1: mass 0.045 -> 0.0482
- link ll_dg_1_2: mass 0.025 -> 0.0164
- link ll_dg_1_3: mass 0.045 -> 0.0362
- link ll_dg_1_4: mass 0.045 -> 0.0505
- link ll_dg_2_1: mass 0.045 -> 0.0546
- link ll_dg_2_2: mass 0.045 -> 0.0362
- link ll_dg_2_3: mass 0.045 -> 0.0362
- link ll_dg_2_4: mass 0.025 -> 0.0266
- link ll_dg_3_1: mass 0.045 -> 0.0526
- link ll_dg_3_2: mass 0.045 -> 0.0362
- link ll_dg_3_3: mass 0.045 -> 0.0362
- link ll_dg_3_4: mass 0.025 -> 0.0266
- link ll_dg_4_1: mass 0.045 -> 0.0548
- link ll_dg_4_2: mass 0.045 -> 0.0362
- link ll_dg_4_3: mass 0.045 -> 0.0362
- link ll_dg_4_4: mass 0.025 -> 0.0266
- link ll_dg_5_1: mass 0.055 -> 0.0744
- link ll_dg_5_2: mass 0.025 -> 0.0164
- link ll_dg_5_3: mass 0.045 -> 0.0362
- link ll_dg_5_4: mass 0.045 -> 0.0505
- link ll_dg_base: mass 0.45 -> 0.51
- link ll_dg_palm: mass 0.35 -> 0.4007

File: dg5f/dg5f_right.urdf (robot description, URDF)
Before this commit: robot dg5f_right, 28 links, 27 joints
Links:
- link rl_dg_1_1: mass 0.045 -> 0.0482
- link rl_dg_1_2: mass 0.025 -> 0.0164
- link rl_dg_1_3: mass 0.045 -> 0.0362
- link rl_dg_1_4: mass 0.045 -> 0.0505
- link rl_dg_2_1: mass 0.045 -> 0.0546
- link rl_dg_2_2: mass 0.045 -> 0.0362
- link rl_dg_2_3: mass 0.045 -> 0.0362
- link rl_dg_2_4: mass 0.025 -> 0.0266
- link rl_dg_3_1: mass 0.045 -> 0.0526
- link rl_dg_3_2: mass 0.045 -> 0.0362
- link rl_dg_3_3: mass 0.045 -> 0.0362
- link rl_dg_3_4: mass 0.025 -> 0.0266
- link rl_dg_4_1: mass 0.045 -> 0.0548
- link rl_dg_4_2: mass 0.045 -> 0.0362
- link rl_dg_4_3: mass 0.045 -> 0.0362
- link rl_dg_4_4: mass 0.025 -> 0.0266
- link rl_dg_5_1: mass 0.055 -> 0.0744
- link rl_dg_5_2: mass 0.025 -> 0.0164
- link rl_dg_5_3: mass 0.045 -> 0.0362
- link rl_dg_5_4: mass 0.045 -> 0.0505
- link rl_dg_base: mass 0.45 -> 0.51
- link rl_dg_palm: mass 0.35 -> 0.4007

Commit message: dg5f update

File: dg5f/dg5f_left.urdf (robot description, URDF)
Before this commit: robot dg5f_left, 28 links, 27 joints
Links:
- link ll_dg_base: mass 0.51 -> 0.3529
- link ll_dg_palm: mass 0.4007 -> 0.5578

File: dg5f/dg5f_left_short.urdf (robot description, URDF)
Before this commit: robot dg5f_left_short, 28 links, 27 joints
Links:
- link ll_dg_base: mass 0.45 -> 0.1112
- link ll_dg_mount: mass 0.05 -> 0.0882
- link ll_dg_palm: mass 0.4007 -> 0.5578

File: dg5f/dg5f_right.urdf (robot description, URDF)
Before this commit: robot dg5f_right, 28 links, 27 joints
Links:
- link rl_dg_base: mass 0.51 -> 0.3529
- link rl_dg_palm: mass 0.4007 -> 0.5578

File: dg5f/dg5f_right_short.urdf (robot description, URDF)
Before this commit: robot dg5f_right_short, 28 links, 27 joints
Links:
- link rl_dg_1_1: mass 0.045 -> 0.0482
- link rl_dg_1_2: mass 0.025 -> 0.0164
- link rl_dg_1_3: mass 0.045 -> 0.0362
- link rl_dg_1_4: mass 0.045 -> 0.0505
- link rl_dg_2_1: mass 0.045 -> 0.0546
- link rl_dg_2_2: mass 0.045 -> 0.0362
- link rl_dg_2_3: mass 0.045 -> 0.0362
- link rl_dg_2_4: mass 0.025 -> 0.0266
- link rl_dg_3_1: mass 0.045 -> 0.0526
- link rl_dg_3_2: mass 0.045 -> 0.0362
- link rl_dg_3_3: mass 0.045 -> 0.0362
- link rl_dg_3_4: mass 0.025 -> 0.0266
- link rl_dg_4_1: mass 0.045 -> 0.0548
- link rl_dg_4_2: mass 0.045 -> 0.0362
- link rl_dg_4_3: mass 0.045 -> 0.0362
- link rl_dg_4_4: mass 0.025 -> 0.0266
- link rl_dg_5_1: mass 0.055 -> 0.0744
- link rl_dg_5_2: mass 0.025 -> 0.0164
- link rl_dg_5_3: mass 0.045 -> 0.0362
- link rl_dg_5_4: mass 0.045 -> 0.0505
- link rl_dg_base: mass 0.45 -> 0.1112
- link rl_dg_mount: mass 0.05 -> 0.0882
- link rl_dg_palm: mass 0.35 -> 0.5578
