Commit message: add dg5f *.xml

File: dg5f/dg5f_left.urdf (robot description, URDF)
Before this commit: robot dg5f_left, 28 links, 27 joints
Joints:
- joint lj_dg_1_tip: origin xyz=0.0 -0.0363 0.0 rpy=0.0 0.0 0.0 -> xyz=0.0 -0.0363 0.0 rpy=0.0 0.0 3.141592653589793

File: dg5f/dg5f_left_short.urdf (robot description, URDF)
Before this commit: robot dg5f_left_short, 28 links, 27 joints
Joints:
- joint lj_dg_1_tip: origin xyz=0.0 -0.0363 0.0 rpy=0.0 0.0 0.0 -> xyz=0.0 -0.0363 0.0 rpy=0.0 0.0 3.141592653589793

File: dg5f/dg5f_right.urdf (robot description, URDF)
Before this commit: robot dg5f_right, 28 links, 27 joints
Joints:
- joint rj_dg_1_tip: origin xyz=0.0 0.0363 0.0 rpy=0.0 0.0 0.0 -> xyz=0.0 0.0363 0.0 rpy=0.0 0.0 3.141592653589793

File: dg5f/dg5f_right_short.urdf (robot description, URDF)
Before this commit: robot dg5f_right_short, 28 links, 27 joints
Joints:
- joint rj_dg_1_tip: origin xyz=0.0 0.0363 0.0 rpy=0.0 0.0 0.0 -> xyz=0.0 0.0363 0.0 rpy=0.0 0.0 3.141592653589793
